File: Ayeeduino_Uno_Rev2/Ayeeduino_Uno_Rev2.kicad_pcb (KiCad board)
At the start: 2 copper layers, 55 x 35 mm, 1 part, among them U1 ATmega328PB-AU

Commit message: working on layout
Parts:
- added C1: 100nF, Capacitor_SMD:C_0603_1608Metric, F.Cu at (78.0, 26.0)
- added C10: 100nF, Capacitor_SMD:C_0603_1608Metric, F.Cu at (68.5, 35.4)
- added C11: 100nF, Capacitor_SMD:C_0603_1608Metric, F.Cu at (72.9, 30.8)
- added C12: 100nF, Capacitor_SMD:C_0603_1608Metric, F.Cu at (72.5, 38.3)
- added C13: 100nF, Capacitor_SMD:C_0603_1608Metric, F.Cu at (80.9, 33.5)
- added C14: 100nF, Capacitor_SMD:C_0603_1608Metric, F.Cu at (82.0, 26.0)
- added C15: 100nF, Capacitor_SMD:C_0603_1608Metric, F.Cu at (81.3, 28.5)
- added C2: 100nF, Capacitor_SMD:C_0603_1608Metric, F.Cu at (82.8, 21.4)
- added C3: 100nF, Capacitor_SMD:C_0603_1608Metric, F.Cu at (85.3, 28.5)
- added C4: 100nF, Capacitor_SMD:C_0603_1608Metric, F.Cu at (80.9, 31.0)
- added C5: 100nF, Capacitor_SMD:C_0603_1608Metric, F.Cu at (76.9, 31.0)
- added C6: 100nF, Capacitor_SMD:C_0603_1608Metric, F.Cu at (90.0, 23.9)
- added C7: 100nF, Capacitor_SMD:C_0603_1608Metric, F.Cu at (86.9, 21.4)
- added C8: 100nF, Capacitor_SMD:C_0603_1608Metric, F.Cu at (72.9, 33.3)
- added C9: 100nF, Capacitor_SMD:C_0603_1608Metric, F.Cu at (76.9, 33.5)
- added F1: 0.5A, Fuse:Fuse_0603_1608Metric_Castellated, F.Cu at (73.1, 28.4)
- added F2: 0.5A, Fuse:Fuse_0603_1608Metric_Castellated, F.Cu at (68.7, 32.9)
- added J1: Conn_01x15, Custom_Vertical_1x_2.54mm_Pin_Header:PinHeader_1x15_P2.54mm_Vertical, F.Cu at (14.0, 44.5)
- added J2: USB_C_Receptacle_USB2.0, Connector_USB:USB_C_Receptacle_XKB_U262-16XN-4BVC11, F.Cu at (15.0, 29.0)
- added J3: Conn_01x15, Custom_Vertical_1x_2.54mm_Pin_Header:PinHeader_1x15_P2.54mm_Vertical, F.Cu at (14.0, 14.0)
- added J4: ICSP, Custom_Vertical_2x_2.54mm_Pin_Header:PinHeader_2x03_P2.54mm_Vertical, F.Cu at (61.6, 32.1)
- added J5: ICSP, Custom_Vertical_2x_2.54mm_Pin_Header:PinHeader_2x03_P2.54mm_Vertical, F.Cu at (61.6, 22.4)
- added R1: 330R, Resistor_SMD:R_0603_1608Metric, F.Cu at (76.5, 38.5)
- added R2: 330R, Resistor_SMD:R_0603_1608Metric, F.Cu at (68.5, 37.9)
- added R3: 330R, Resistor_SMD:R_0603_1608Metric, F.Cu at (90.9, 21.4)
- added R4: 5.1K, Resistor_SMD:R_0603_1608Metric, F.Cu at (72.5, 35.8)
- added R5: 5.1K, Resistor_SMD:R_0603_1608Metric, F.Cu at (77.3, 28.5)
- added R6: 1M, Resistor_SMD:R_0603_1608Metric, F.Cu at (84.9, 31.0)
- added R7: 1M, Resistor_SMD:R_0603_1608Metric, F.Cu at (76.5, 36.0)
- added SW1: RST, Button_Switch_SMD:SW_SPST_TL3342, F.Cu at (71.2, 23.6)
- added U2: ME6212, Package_TO_SOT_SMD:SOT-23-5, F.Cu at (78.4, 22.4)
- added U3: LED_RGB_0603_R6GHBHC-C01-2T, Custom_Parts:LED_DUAL_0603, F.Cu at (86.0, 24.5)
- added U4: XC6206P332MR, Package_TO_SOT_SMD:SOT-23, F.Cu at (68.7, 29.4)
- added U5: CH340G, Package_SO:SOIC-16_3.9x9.9mm_P1.27mm, F.Cu at (28.0, 29.0)
- added Y1: 16MHz, Crystal:Crystal_SMD_3225-4Pin_3.2x2.5mm, F.Cu at (37.5, 34.8)
- added Y2: 12MHz, Crystal:Crystal_SMD_3225-4Pin_3.2x2.5mm, F.Cu at (26.9, 36.1)
- moved U1 10.4 mm to (43.0, 29.0)
Connections:
- net Net-(U1-Pad21) renamed GNDREF
- U1 pad 1: Net-(U1-Pad1) -> /D3
- U1 pad 10: Net-(U1-Pad10) -> /D6
- U1 pad 11: Net-(U1-Pad11) -> /D7
- U1 pad 12: Net-(U1-Pad12) -> /D8
- U1 pad 13: Net-(U1-Pad13) -> /D9
- U1 pad 14: Net-(U1-Pad14) -> /D10_SS0
- U1 pad 15: Net-(U1-Pad15) -> /D11_MOSI0_TX1
- U1 pad 16: Net-(U1-Pad16) -> /D12_MISO0_RX1
- U1 pad 17: Net-(U1-Pad17) -> /D13_SCK0
- U1 pad 18: Net-(U1-Pad18) -> +5V
- U1 pad 19: Net-(U1-Pad19) -> /ADC6_SS1
- U1 pad 2: Net-(U1-Pad2) -> /D4
- U1 pad 20: Net-(U1-Pad20) -> /AREF
- U1 pad 22: Net-(U1-Pad22) -> /ADC7_MOSI1
- U1 pad 23: Net-(U1-Pad23) -> /ADC0_MISO1
- U1 pad 24: Net-(U1-Pad24) -> /ADC1_SCK1
- U1 pad 25: Net-(U1-Pad25) -> /ADC2
- U1 pad 26: Net-(U1-Pad26) -> /ADC3
- U1 pad 27: Net-(U1-Pad27) -> /ADC4_SDA0
- U1 pad 28: Net-(U1-Pad28) -> /ADC5_SCL0
- U1 pad 29: Net-(U1-Pad29) -> /RST
- U1 pad 3: Net-(U1-Pad3) -> /SDA1
- U1 pad 30: Net-(U1-Pad30) -> /D0_RX0
- U1 pad 31: Net-(U1-Pad31) -> /D1_TX0
- U1 pad 32: Net-(U1-Pad32) -> /D2
- U1 pad 4: Net-(U1-Pad4) -> +5V
- U1 pad 6: Net-(U1-Pad6) -> /SCL1
- U1 pad 9: Net-(U1-Pad9) -> /D5
Routing:
- net /D0_RX0: track 0.00 -> 20.6 mm
- net /D1_TX0: track 0.00 -> 17.8 mm
- net /D3: track 0.00 -> 12.3 mm
- net /D-: track 0.00 -> 10.9 mm, vias 0 -> 2
- net /D+: track 0.00 -> 9.74 mm
- net Net-(C10-Pad1): track 0.00 -> 6.12 mm
- net Net-(C12-Pad1): track 0.00 -> 4.30 mm
- net Net-(C13-Pad1): track 0.00 -> 4.27 mm
- net Net-(C9-Pad1): track 0.00 -> 2.06 mm
Other:
- board size 55 x 35 mm -> 40 x 34.5 mm
- net class Default: clearance 0.2 -> 0.127; trace_width 0.25 -> 0.127; via_dia 0.8 -> 0.6; via_drill 0.4 -> 0.35
- rule trace_clearance: 0.2 -> 0.127
- rule trace_min: 0.2 -> 0.1016
- rule via_min_size: 0.4 -> 0.3
