File: Ayeeduino_Uno_Rev2/Ayeeduino_Uno_Rev2.kicad_sch (KiCad schematic)
At the start: 27 parts, among them U1 ATmega328PB-AU

Commit message: working on layout
Parts:
- removed Q?: FDN360P, Package_TO_SOT_SMD:SOT-23, symbol Device:Q_PMOS_GSD
- removed Y?: Crystal_GND24_Small, symbol Device:Crystal_GND24_Small
- added C10, C14, C15, C9: 100nF, Capacitor_SMD:C_0603_1608Metric, symbol Device:C_Small
- added F2: 0.5A, Fuse:Fuse_0603_1608Metric_Castellated, symbol Device:Fuse_Small
- added J1, J3: Conn_01x15, Custom_Vertical_1x_2.54mm_Pin_Header:PinHeader_1x15_P2.54mm_Vertical, symbol Connector_Generic:Conn_01x15
- added J4, J5: ICSP, Custom_Vertical_2x_2.54mm_Pin_Header:PinHeader_2x03_P2.54mm_Vertical, symbol Connector_Generic:Conn_02x03_Odd_Even
- added R6: 1M, Resistor_SMD:R_0603_1608Metric, symbol Device:R_Small_US
- added SW1: RST, Button_Switch_SMD:SW_SPST_TL3342, symbol Switch:SW_Push_45deg
- added Y1: 16MHz, Crystal:Crystal_SMD_3225-4Pin_3.2x2.5mm, symbol Device:Crystal_GND24_Small
- F1: renamed from F?; footprint (none) -> Fuse:Fuse_0603_1608Metric_Castellated
- gave numbers to parts that had none: 23
Connections:
- net RX is gone; now on net D1_TX0: R1.2, U5.3 (RXD)
- net TX is gone; now on net D0_RX0: R3.2, U5.2 (TXD)
- net VUSBF is gone; now on net VBUS: F1.2
- net +3V3: now also J5.3 (Pin_3)
- net +5V: now also U1.18 (AVCC), U1.4 (VCC), C14.1, C15.1, J1.14 (Pin_14), J3.14 (Pin_14), J4.2 (Pin_2), J5.1 (Pin_1), J5.4 (Pin_4)
- net ADC2: now also J1.9 (Pin_9)
- net ADC3: now also J1.10 (Pin_10)
- net AREF: now also J3.13 (Pin_13)
- net D2: now also J3.3 (Pin_3)
- net D3: now also J3.4 (Pin_4)
- net D4: now also J3.5 (Pin_5)
- net D5: now also J3.6 (Pin_6)
- net D6: now also J3.7 (Pin_7)
- net D7: now also J3.8 (Pin_8)
- net D8: now also J1.1 (Pin_1)
- net D9: now also J1.2 (Pin_2)
- net GNDREF: now also U1.21 (GND), U1.5 (GND), U5.1 (GND), C10.2, C14.2, C15.2, C9.2, J1.15 (Pin_15), J3.15 (Pin_15), J4.6 (Pin_6), J5.5 (Pin_5), J5.6 (Pin_6), SW1.2, Y1.1, Y1.3
- net RST: now also J1.13 (Pin_13), J4.5 (Pin_5), SW1.1
- net VBUS: now also F2.2
- net ADC6_SS1: now reaches U1.19 (PE2)
- net ADC6_SS1: now also J3.11 (Pin_11)
- net ADC7_MOSI1: now reaches U1.22 (PE3)
- net ADC7_MOSI1: now also J3.12 (Pin_12)
- net SDA1: now reaches U1.3 (PE0)
- net SDA1: now also J3.9 (Pin_9)
- net SCL1: now reaches U1.6 (PE1)
- net SCL1: now also J3.10 (Pin_10)
- net at U1.7 (XTAL1/PB6): now also C10.1, R6.1, Y1.2
- net at U1.8 (XTAL2/PB7): now also C9.1, R6.2, Y1.4
- net ADC0 renamed ADC0_MISO1
- net ADC0_MISO1: now also J1.7 (Pin_7)
- net ADC1 renamed ADC1_SCK1
- net ADC1_SCK1: now also J1.8 (Pin_8)
- net ADC4_SDA renamed ADC4_SDA0
- net ADC4_SDA0: now also J1.11 (Pin_11)
- net ADC5_SCL renamed ADC5_SCL0
- net ADC5_SCL0: now also J1.12 (Pin_12)
- net D0 renamed D0_RX0
- net D0_RX0: now also J3.1 (Pin_1)
- net D1 renamed D1_TX0
- net D1_TX0: now also J3.2 (Pin_2)
- net D10 renamed D10_SS0
- net D10_SS0: now also J1.3 (Pin_3)
- net D11 renamed D11_MOSI0_TX1
- net D11_MOSI0_TX1: now also J1.4 (Pin_4), J4.4 (Pin_4)
- net D12 renamed D12_MISO0_RX1
- net D12_MISO0_RX1: now also J1.5 (Pin_5), J4.1 (Pin_1)
- net D13 renamed D13_SCK0
- net D13_SCK0: now also J1.6 (Pin_6), J4.3 (Pin_3)
- new net: F2.1, J5.2 (Pin_2)
