File: QFP_Programmers/AtMega328P_Programmer/AtMega328P_Programmer.kicad_pcb (KiCad board)
At the start: 2 copper layers, 50 x 50 mm, 15 parts, among them J1 ICSP, U1 ATmega328P-AU, Y1 16MHz

Commit message: Macro_Keys Layout complete + Programmer WIP
Parts:
- removed the U1 at (37.0, 37.0) (x2)
- added U1: ATmega328P-AU, Package_QFP:TQFP-32_7x7mm_P0.8mm, B.Cu at (37.0, 37.0)
- added U1: ATmega328P-AU, Package_QFP:TQFP-32_7x7mm_P0.8mm, F.Cu at (37.0, 37.0)
Other:
- net class Default removed
